File: controller/controller.kicad_pcb (KiCad board)
At the start: 2 copper layers, 69.6 x 37.3 mm, 50 parts, among them J1 Conn_01x25_Membrane, J2 Conn_01x04, J3 Conn_Solenoid_Driver, J4 Conn_01x04, J5 Conn_01x07, J6 Conn_01x06, SW1 SW_Push, SW2 SW_Push, U1 AMS1117-3.3, U2 STM32F303RCT6, U3 TPS2553DBVR, U4 USBLC6-2SC6, Y1 16MHz

Commit message: Added version 1.0b, and exported 3mm version gerber
Parts:
- removed J4: Conn_01x04, Connector_PinHeader_2.54mm:PinHeader_1x04_P2.54mm_Vertical
- added C18: 4.7uF, Capacitor_SMD:C_0805_2012Metric_Pad1.15x1.40mm_HandSolder, F.Cu at (110.0, 155.8)
- added R10: 62k, Resistor_SMD:R_0805_2012Metric_Pad1.15x1.40mm_HandSolder, F.Cu at (118.9, 157.2)
- added R11: 62k, Resistor_SMD:R_0805_2012Metric_Pad1.15x1.40mm_HandSolder, F.Cu at (96.9, 156.3)
- added R12: 62k, Resistor_SMD:R_0805_2012Metric_Pad1.15x1.40mm_HandSolder, F.Cu at (114.8, 157.2)
- added R9: 62k, Resistor_SMD:R_0805_2012Metric_Pad1.15x1.40mm_HandSolder, F.Cu at (81.9, 138.3)
- R6: value 1.5k -> 62k
- U2: value STM32F303RCT6 -> STM32F446RETx
- moved R6 9.77 mm to (108.6, 134.9), turned to 180 degrees
- moved R4 2.43 mm to (105.1, 135.3)
- moved R3 2.26 mm to (102.8, 135.3)
- moved R5 2.11 mm to (112.8, 134.9)
Connections:
- net MEMBRANE19 renamed MEMBRANE19_PA5
- net Net-(C10-Pad2) renamed /NRST
- net Net-(C8-Pad1) renamed /OSCI
- net Net-(C9-Pad1) renamed /OSCO_RES
- net Net-(R1-Pad2) renamed /OSCO
- net Net-(R2-Pad1) renamed /BOOT0
- net SOLENOID_TRIGGER renamed SOLENOID_TRIGGER_CAN_RX_BL
- J1 pad 1: MEMBRANE1 -> MEMBRANE1_PA10
- J1 pad 4: MEMBRANE4 -> MEMBRANE4_PC9
- J1 pad 6: MEMBRANE6 -> MEMBRANE6_PC7
- J5 pad 6: GPIO_PC3 -> Net-(J5-Pad6)
- R4 pad 2: LEDDRV2 -> LEDDRV2_USART3RX_BL
- R6 pad 1: +3.3VA -> GND
- R6 pad 2: USB_DP -> LEDDRV2_USART3RX_BL
- R8 pad 2: UART_RX -> MEMBRANE1_PA10
- U2 pad 10: MEMBRANE25 -> MEMBRANE24
- U2 pad 11: GPIO_PC3 -> MEMBRANE25
- U2 pad 18: MEMBRANE22 -> GND
- U2 pad 28: MEMBRANE12 -> GND
- U2 pad 29: MEMBRANE11 -> MEMBRANE12
- U2 pad 30: MEMBRANE10 -> Net-(C18-Pad1)
- U2 pad 33: MEMBRANE9 -> MEMBRANE11
- U2 pad 34: MEMBRANE8 -> MEMBRANE10
- U2 pad 35: MEMBRANE7 -> MEMBRANE9
- U2 pad 36: MEMBRANE6 -> MEMBRANE8
- U2 pad 37: MEMBRANE5 -> MEMBRANE7
- U2 pad 38: MEMBRANE4 -> MEMBRANE6_PC7
- U2 pad 39: MEMBRANE3 -> MEMBRANE5
- U2 pad 40: MEMBRANE2 -> MEMBRANE4_PC9
- U2 pad 41: MEMBRANE1 -> MEMBRANE3
- U2 pad 42: UART_TX -> MEMBRANE2
- U2 pad 43: UART_RX -> MEMBRANE1_PA10
- U2 pad 52: LEDDRV2 -> LEDDRV2_USART3RX_BL
- U2 pad 58: Net-(U2-Pad58) -> GND
- U2 pad 62: Net-(U2-Pad62) -> GND
- U2 pad 8: MEMBRANE23 -> MEMBRANE22
- U2 pad 9: MEMBRANE24 -> MEMBRANE23
Routing:
- net MEMBRANE1: track 28.5 -> 0.00 mm, vias 1 -> 0
- net MEMBRANE1_PA10: track 0.00 -> 26.6 mm, vias 0 -> 1
- net GPIO_PC3: track 24.4 -> 0.00 mm
- net MEMBRANE4_PC9: track 0.00 -> 23.9 mm, vias 0 -> 1
- net MEMBRANE4: track 21.5 -> 0.00 mm, vias 1 -> 0
- net MEMBRANE6_PC7: track 0.00 -> 20.5 mm, vias 0 -> 1
- net +3.3VA: track 156.3 -> 174.2 mm, vias 6 -> 9
- net MEMBRANE6: track 17.8 -> 0.00 mm, vias 1 -> 0
- net UART_RX: track 16.1 -> 0.00 mm
- net UART_TX: track 12.1 -> 0.00 mm
- net LEDDRV2_USART3RX_BL: track 0.00 -> 9.16 mm
- net MEMBRANE10: track 14.5 -> 21.5 mm
- net SOLENOID_TRIGGER_CAN_RX_BL: track 21.2 -> 28.0 mm
- net MEMBRANE11: track 15.8 -> 22.5 mm
- net MEMBRANE22: track 32.5 -> 39.0 mm
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Other:
- board text added: "3mm holes"
- board text added: "OverNumpadController Rev. 1.0b"
- board text removed: "OverNumpadController Rev. 1.0"
- board text removed: "PC3"
- board text removed: "RX/PA10"
- board text removed: "TX/PA9"
- board text removed: "UART"

Commit message: Added v1.1b version
Parts:
- removed J5: Conn_01x07, Connector_PinHeader_2.54mm:PinHeader_1x07_P2.54mm_Vertical
- removed SW2: SW_Push, controller:TS342A2PWZ
- added C19: 100nF, Capacitor_SMD:C_0805_2012Metric_Pad1.15x1.40mm_HandSolder, F.Cu at (75.8, 152.2)
- added C20: 1uF, Capacitor_SMD:C_0805_2012Metric_Pad1.15x1.40mm_HandSolder, F.Cu at (82.5, 141.8)
- added J4: Conn_01x01, controller:PinHeader_1x01_P1.27mm_Vertical_mod_no_courtyard_no_ref, F.Cu at (115.8, 137.7)
- added Q1: Q_PMOS_GSD AO3401A, Package_TO_SOT_SMD:SOT-23, F.Cu at (76.0, 146.1)
- added Q2: Q_NMOS_GSD 2N7002, Package_TO_SOT_SMD:SOT-23, F.Cu at (87.7, 148.4)
- added Q3: Q_NMOS_GSD 2N7002, Package_TO_SOT_SMD:SOT-23, F.Cu at (71.0, 149.4)
- added R13: 2k, Resistor_SMD:R_0805_2012Metric_Pad1.15x1.40mm_HandSolder, F.Cu at (81.2, 155.1)
- added R14: 2k, Resistor_SMD:R_0805_2012Metric_Pad1.15x1.40mm_HandSolder, F.Cu at (84.3, 155.1)
- added R15: 2k, Resistor_SMD:R_0805_2012Metric_Pad1.15x1.40mm_HandSolder, F.Cu at (87.5, 155.1)
- added R16: 390, Resistor_SMD:R_0805_2012Metric_Pad1.15x1.40mm_HandSolder, F.Cu at (79.3, 141.8)
- added R17: 2k, Resistor_SMD:R_0805_2012Metric_Pad1.15x1.40mm_HandSolder, F.Cu at (87.7, 151.7)
- added R18: 2k, Resistor_SMD:R_0805_2012Metric_Pad1.15x1.40mm_HandSolder, F.Cu at (76.3, 149.6)
- added U5: 24LC64, Package_SO:SOIC-8_3.9x4.9mm_P1.27mm, F.Cu at (74.7, 156.3)
- JP1: value SolderJumper_2_Open -> SolderJumper_2_Bridged; footprint controller:shortable -> controller:shortable_shorted
- SW1: footprint controller:TS342A2PWZ -> controller:switch_K2-1187SQ-A4SW-06
- moved C10 9.10 mm to (90.7, 148.4), turned to 90 degrees
- moved SW1 6.09 mm to (82.2, 148.3), turned to 270 degrees
- moved R2 2.47 mm to (85.7, 141.8), turned to 270 degrees
- moved J6 1.92 mm to (107.7, 137.7)
Connections:
- net Net-(C18-Pad1) renamed /VCAP_1
- net Net-(D1-Pad1) renamed /TopLightsGround
- net Net-(D1-Pad2) renamed /LD1R
- net Net-(D2-Pad2) renamed /LD2R
- net Net-(D3-Pad2) renamed /LD3R
- net Net-(D4-Pad1) renamed /BottomLightsGround
- SW1 pad 2: /BOOT0 -> Net-(SW1-Pad2)
Routing:
- net VBUS: track 113.2 -> 65.2 mm
- net Net-(Q2-Pad1): track 0.00 -> 21.5 mm
- net /TopLightsGround: track 48.2 -> 58.2 mm
- net /BottomLightsGround: track 64.8 -> 72.2 mm
- net /NRST: track 21.3 -> 14.3 mm
- net /LD2R: track 57.3 -> 63.7 mm
- net Net-(Q1-Pad1): track 0.00 -> 5.96 mm
- net /BOOT0_DRV: track 0.00 -> 4.88 mm
- net LEDDRV3: track 7.27 -> 12.0 mm
- net /BOOT0: track 25.0 -> 29.7 mm
- net +3.3VA: track 174.2 -> 169.6 mm, vias 9 -> 7
- net GPIO_PA2: track 22.1 -> 26.6 mm
- net GPIO_PA0: track 31.6 -> 27.6 mm
- net /LD3R: track 31.8 -> 29.2 mm
- net /LD1R: track 40.5 -> 42.3 mm
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Other:
- board text added: "3.2mm holes"
- board text added: "OverNumpadController Rev. 1.1b"
- board text added: "RST & PROG"
- board text removed: "3mm holes"
- board text removed: "OverNumpadController Rev. 1.0b"
- board text removed: "PA0"
- board text removed: "PA1"
- board text removed: "PA2"
- board text removed: "PROG"
- board text removed: "RST"
