File: controller/controller.sch (KiCad schematic (older format))
At the start: 65 parts, among them J1 Conn_01x25_Membrane, J2 Conn_01x04, J3 Conn_Solenoid_Driver, J4 Conn_01x01, J6 Conn_01x06, Q1 Q_PMOS_GSD AO3401A, Q2 Q_NMOS_GSD 2N7002, Q3 Q_NMOS_GSD 2N7002, SW1 SW_Push, U1 AMS1117-3.3, U2 STM32F446RETx, U3 TPS2553DBVR, U4 USBLC6-2SC6, U5 24LC64, Y1 16MHz

Commit message: Replaced out-of-stock part
Parts:
- C8, C9: LCSC C1785 -> C157608
Changed lines of the file:
@@
 F 2 "Capacitor_SMD:C_0805_2012Metric_Pad1.15x1.40mm_HandSolder" H 2413 3400 50  0001 C CNN
 F 3 "~" H 2375 3550 50  0001 C CNN
-F 4 "C1785" H 2375 3550 50  0001 C CNN "LCSC"
+F 4 "C157608" H 2375 3550 50  0001 C CNN "LCSC"
 	1    2375 3550
 	0    1    1    0
@@
 F 2 "Capacitor_SMD:C_0805_2012Metric_Pad1.15x1.40mm_HandSolder" H 2413 3850 50  0001 C CNN
 F 3 "~" H 2375 4000 50  0001 C CNN
-F 4 "C1785" H 2375 4000 50  0001 C CNN "LCSC"
+F 4 "C157608" H 2375 4000 50  0001 C CNN "LCSC"
 	1    2375 4000
 	0    1    1    0
